Commit message: Improved robot model

File: holly_tf/holly.urdf (robot description, URDF)
Before this commit: robot holly, 5 links, 4 joints
Links:
- added link /wheel1; visual cylinder length=0.06 radius=0.06
- added link /wheel2; visual cylinder length=0.06 radius=0.06
- added link /wheel3; visual cylinder length=0.06 radius=0.06
- added link /wheel4; visual cylinder length=0.06 radius=0.06
- added link /wheel5; visual cylinder length=0.06 radius=0.06
- added link /wheel6; visual cylinder length=0.06 radius=0.06
- link /base_link: geometry visual box size=0.505 0.27 0.02

Commit message: fixed wheels

File: holly_tf/holly.urdf (robot description, URDF)
Before this commit: robot holly, 11 links, 4 joints
Joints:
- added joint base_to_wheel1: type fixed, parent /base_link, child /wheel1
- added joint base_to_wheel2: type fixed, parent /base_link, child /wheel2
- added joint base_to_wheel3: type fixed, parent /base_link, child /wheel3
- added joint base_to_wheel4: type fixed, parent /base_link, child /wheel4
- added joint base_to_wheel5: type fixed, parent /base_link, child /wheel5
- added joint base_to_wheel6: type fixed, parent /base_link, child /wheel6

Commit message: Updated wheels

File: holly_tf/holly.urdf (robot description, URDF)
Before this commit: robot holly, 11 links, 10 joints
Links:
- added link /motor1; visual cylinder length=0.075 radius=0.016
- added link /motor2; visual cylinder length=0.075 radius=0.016
- added link /motor3; visual cylinder length=0.075 radius=0.016
- added link /motor4; visual cylinder length=0.075 radius=0.016
- added link /motor5; visual cylinder length=0.075 radius=0.016
- added link /motor6; visual cylinder length=0.075 radius=0.016
Joints:
- removed joint base_to_wheel1
- removed joint base_to_wheel2
- removed joint base_to_wheel3
- removed joint base_to_wheel4
- removed joint base_to_wheel5
- removed joint base_to_wheel6
- added joint base_to_motor1: type continuous, parent /base_link, child /motor1, origin xyz=0 0.17 0.06 rpy=1.570895 0 0, axis 0 1 0
- added joint base_to_motor2: type continuous, parent /base_link, child /motor2, origin xyz=0 -0.17 0.06 rpy=1.570895 3.14159 0, axis 0 1 0
- added joint base_to_motor3: type continuous, parent /base_link, child /motor3, origin xyz=0.23 -0.17 0.06 rpy=1.570895 3.14159 0, axis 0 1 0
- added joint base_to_motor4: type continuous, parent /base_link, child /motor4, origin xyz=0.23 0.17 0.06 rpy=1.570895 0 0, axis 0 1 0
- added joint base_to_motor5: type continuous, parent /base_link, child /motor5, origin xyz=-0.23 -0.17 0.06 rpy=1.570895 3.14159 0, axis 0 1 0
- added joint base_to_motor6: type continuous, parent /base_link, child /motor6, origin xyz=-0.23 0.17 0.06 rpy=1.570895 0 0, axis 0 1 0
- added joint motor_to_wheel1: type continuous, parent /motor1, child /wheel1, origin xyz=0 0 0 rpy=0 0 0, axis 0 0 1
- added joint motor_to_wheel2: type continuous, parent /motor2, child /wheel2, origin xyz=0 0 0 rpy=0 0 0, axis 0 0 1
- added joint motor_to_wheel3: type continuous, parent /motor3, child /wheel3, origin xyz=0 0 0 rpy=0 0 0, axis 0 0 1
- added joint motor_to_wheel4: type continuous, parent /motor4, child /wheel4, origin xyz=0 0 0 rpy=0 0 0, axis 0 0 1
- added joint motor_to_wheel5: type continuous, parent /motor5, child /wheel5, origin xyz=0 0 0 rpy=0 0 0, axis 0 0 1
- added joint motor_to_wheel6: type continuous, parent /motor6, child /wheel6, origin xyz=0 0 0 rpy=0 0 0, axis 0 0 1

Commit message: updates to the model

File: holly_tf/holly.urdf (robot description, URDF)
Before this commit: robot holly, 17 links, 16 joints
Links:
- removed link /motor1
- removed link /motor2
- removed link /motor3
- removed link /motor4
- removed link /motor5
- removed link /motor6
- added link /bogie_left; visual box size=0.32 0.02 0.02
- added link /bogie_rear; visual box size=0.38 0.02 0.02
- added link /bogie_right; visual box size=0.32 0.02 0.02
- link /kinect_depth_frame: mass 0.0001 -> None
- link /kinect_depth_optical_frame: mass 0.0001 -> None
- link /kinect_link: mass 0.0001 -> None
Joints:
- removed joint base_to_motor1
- removed joint base_to_motor2
- removed joint base_to_motor3
- removed joint base_to_motor4
- removed joint base_to_motor5
- removed joint base_to_motor6
- removed joint motor_to_wheel1
- removed joint motor_to_wheel2
- removed joint motor_to_wheel3
- removed joint motor_to_wheel4
- removed joint motor_to_wheel5
- removed joint motor_to_wheel6
- added joint base_to_bogie_left: type continuous, parent /base_link, child /bogie_left, origin xyz=0.12 0.17 0 rpy=0 0 0, axis 0 1 0, limit lower=-0.261 upper=0.261
- added joint base_to_bogie_rear: type continuous, parent /base_link, child /bogie_rear, origin xyz=-0.27 0 0 rpy=0 0 0, axis 1 0 0, limit lower=-0.261 upper=0.261
- added joint base_to_bogie_right: type continuous, parent /base_link, child /bogie_right, origin xyz=0.12 -0.17 0 rpy=0 0 0, axis 0 1 0, limit lower=-0.261 upper=0.261
- added joint bogie_left_to_motor1: type continuous, parent /bogie_left, child /wheel1, origin xyz=0.1 0.0 -0.08 rpy=1.570895 0 0, axis 0 1 0, limit lower=-0.785 upper=0.785
- added joint bogie_left_to_motor2: type fixed, parent /bogie_left, child /wheel2, origin xyz=-0.1 0.0 -0.08 rpy=1.570895 0 0, axis 0 1 0
- added joint bogie_rear_to_motor5: type continuous, parent /bogie_rear, child /wheel5, origin xyz=0 0.17 -0.08 rpy=1.570895 0 0, axis 0 1 0, limit lower=-0.785 upper=0.785
- added joint bogie_rear_to_motor6: type continuous, parent /bogie_rear, child /wheel6, origin xyz=0 -0.17 -0.08 rpy=1.570895 3.14159 0, axis 0 1 0, limit lower=-0.785 upper=0.785
- added joint bogie_right_to_motor3: type continuous, parent /bogie_right, child /wheel3, origin xyz=0.1 0 -0.08 rpy=1.570895 3.14159 0, axis 0 1 0, limit lower=-0.785 upper=0.785
- added joint bogie_right_to_motor4: type fixed, parent /bogie_right, child /wheel4, origin xyz=-0.1 0 -0.08 rpy=1.570895 3.14159 0, axis 0 1 0

Commit message: model fixes

File: holly_tf/holly.urdf (robot description, URDF)
Before this commit: robot holly, 14 links, 13 joints
Joints:
- joint base_to_bogie_left: type continuous -> revolute
- joint base_to_bogie_rear: type continuous -> revolute
- joint base_to_bogie_right: type continuous -> revolute
- joint bogie_left_to_motor1: type continuous -> revolute
- joint bogie_rear_to_motor5: type continuous -> revolute
- joint bogie_rear_to_motor6: type continuous -> revolute
- joint bogie_right_to_motor3: type continuous -> revolute

Commit message: fixes

File: holly_tf/holly.urdf (robot description, URDF)
Before this commit: robot holly, 14 links, 13 joints
Joints:
- joint base_to_bogie_left: limit lower=-0.261 upper=0.261 -> lower=-0.261 upper=0.261 effort=1000 velocity=0.5
- joint base_to_bogie_rear: limit lower=-0.261 upper=0.261 -> lower=-0.261 upper=0.261 effort=1000 velocity=0.5
- joint base_to_bogie_right: limit lower=-0.261 upper=0.261 -> lower=-0.261 upper=0.261 effort=1000 velocity=0.5
- joint bogie_left_to_motor1: limit lower=-0.785 upper=0.785 -> lower=-0.785 upper=0.785 effort=1000 velocity=0.5
- joint bogie_rear_to_motor5: limit lower=-0.785 upper=0.785 -> lower=-0.785 upper=0.785 effort=1000 velocity=0.5
- joint bogie_rear_to_motor6: limit lower=-0.785 upper=0.785 -> lower=-0.785 upper=0.785 effort=1000 velocity=0.5
- joint bogie_right_to_motor3: limit lower=-0.785 upper=0.785 -> lower=-0.785 upper=0.785 effort=1000 velocity=0.5

Commit message: no message

File: holly_tf/holly.urdf (robot description, URDF)
Before this commit: robot holly, 14 links, 13 joints
Links:
- added link /chassis_height_sensor; visual box size=0.05 0.05 0.05
Joints:
- added joint base_to_chassis_height_sensor: type fixed, parent /base_link, child /chassis_height_sensor, origin xyz=0 0.0 0.0 rpy=0 1.570895 0

Commit message: no message

File: holly_tf/holly.urdf (robot description, URDF)
Before this commit: robot holly, 15 links, 14 joints
Links:
- added link /base_footprint; visual box size=0.64 0.35 0.005
Joints:
- joint base_to_bogie_left: origin xyz=0.12 0.17 0 rpy=0 0 0 -> xyz=0.12 0.17 -0.03 rpy=0 0 0
- joint base_to_bogie_rear: origin xyz=-0.27 0 0 rpy=0 0 0 -> xyz=-0.27 0 -0.03 rpy=0 0 0
- joint base_to_bogie_right: origin xyz=0.12 -0.17 0 rpy=0 0 0 -> xyz=0.12 -0.17 -0.03 rpy=0 0 0

Commit message: no message

File: holly_tf/holly.urdf (robot description, URDF)
Before this commit: robot holly, 16 links, 14 joints
Joints:
- added joint base_to_footprint: type fixed, parent /base_footprint, child /base_link, origin xyz=0 0 0.21 rpy=0 0 0

Commit message: no message

File: holly_tf/holly.urdf (robot description, URDF)
Before this commit: robot holly, 16 links, 15 joints
Joints:
- joint base_to_kinect_sensor: origin xyz=0.25 0.0 0.38 rpy=0 0.349066 0 -> xyz=0.25 0.0 0.38 rpy=0 0.261799 0

Commit message: no message

File: holly_tf/holly.urdf (robot description, URDF)
Before this commit: robot holly, 16 links, 15 joints
Joints:
- joint base_to_laserscan_sensor: origin xyz=0.25 0.0 0.0 rpy=0 0 0 -> xyz=0.32 0.0 0.0 rpy=0 0 0; parent /base_link -> /base_footprint

Commit message: Lowered the height of the sensor

File: holly_tf/holly.urdf (robot description, URDF)
Before this commit: robot holly, 16 links, 15 joints
Joints:
- joint base_to_kinect_sensor: origin xyz=0.25 0.0 0.38 rpy=0 0.261799 0 -> xyz=0.25 0.0 0.34 rpy=0 0.261799 0

Commit message: no message

File: holly_tf/holly.urdf (robot description, URDF)
Before this commit: robot holly, 16 links, 15 joints
Joints:
- joint base_to_laserscan_sensor: parent /base_footprint -> /base_link

Commit message: no message

File: holly_tf/holly.urdf (robot description, URDF)
Before this commit: robot holly, 16 links, 15 joints
Links:
- removed link /base_footprint
Joints:
- removed joint base_to_footprint

Commit message: no message

File: holly_tf/holly.urdf (robot description, URDF)
Before this commit: robot holly, 15 links, 14 joints
Joints:
- joint base_to_laserscan_sensor: origin xyz=0.32 0.0 0.0 rpy=0 0 0 -> xyz=0.32 0.0 -0.2 rpy=0 0 0

Commit message: /base_footprint

File: holly_tf/holly.urdf (robot description, URDF)
Before this commit: robot holly, 15 links, 14 joints
Links:
- added link /base_footprint; visual box size=0.65 0.38 0.01

Commit message: no message

File: holly_tf/holly.urdf (robot description, URDF)
Before this commit: robot holly, 16 links, 14 joints
Joints:
- added joint base_to_base_footprint: type fixed, parent /base_link, child /base_footprint, origin xyz=0 0 -0.2

Commit message: remove laserscan offset

File: holly_tf/holly.urdf (robot description, URDF)
Before this commit: robot holly, 16 links, 15 joints
Joints:
- joint base_to_laserscan_sensor: origin xyz=0.32 0.0 -0.2 rpy=0 0 0 -> xyz=0.32 0.0 0 rpy=0 0 0

Commit message: no message

File: holly_tf/holly.urdf (robot description, URDF)
Before this commit: robot holly, 16 links, 15 joints
Joints:
- joint base_to_laserscan_sensor: origin xyz=0.32 0.0 0 rpy=0 0 0 -> xyz=0.32 0.0 -0.2 rpy=0 0 0

Commit message: no message

File: holly_tf/holly.urdf (robot description, URDF)
Before this commit: robot holly, 16 links, 15 joints
Joints:
- joint base_to_laserscan_sensor: origin xyz=0.32 0.0 -0.2 rpy=0 0 0 -> xyz=0.32 0.0 0.0 rpy=0 0 0; parent /base_link -> /base_footprint

Commit message: Moved the range sensor

File: holly_tf/holly.urdf (robot description, URDF)
Before this commit: robot holly, 16 links, 15 joints
Links:
- removed link /chassis_height_sensor
- added link /front_distance_sensor; visual box size=0.05 0.05 0.05
Joints:
- removed joint base_to_chassis_height_sensor
- added joint base_to_front_distance_sensor: type fixed, parent /base_link, child /front_distance_sensor, origin xyz=0.32 0.0 0.0 rpy=0 0 0

Commit message: no message

File: holly_tf/holly.urdf (robot description, URDF)
Before this commit: robot holly, 16 links, 15 joints
Links:
- link /front_distance_sensor: geometry visual box size=0.02 0.02 0.02
Joints:
- joint base_to_front_distance_sensor: origin xyz=0.32 0.0 0.0 rpy=0 0 0 -> xyz=0.22 0.0 -0.04 rpy=0 0 0

Commit message: no message

File: holly_tf/holly.urdf (robot description, URDF)
Before this commit: robot holly, 16 links, 15 joints
Links:
- added link /rear_distance_sensor; visual box size=0.02 0.02 0.02
Joints:
- added joint base_to_rear_distance_sensor: type fixed, parent /base_link, child /rear_distance_sensor, origin xyz=-0.22 0.0 -0.04 rpy=0 0 3.14159

Commit message: no message

File: holly_tf/holly.urdf (robot description, URDF)
Before this commit: robot holly, 17 links, 16 joints
Joints:
- joint base_to_rear_distance_sensor: origin xyz=-0.22 0.0 -0.04 rpy=0 0 3.14159 -> xyz=-0.27 0.0 -0.04 rpy=0 0 3.14159

Commit message: Range sensor updates

File: holly_tf/holly.urdf (robot description, URDF)
Before this commit: robot holly, 17 links, 16 joints
Links:
- removed link /front_distance_sensor
- added link /front_left_distance_sensor; visual box size=0.02 0.02 0.02
- added link /front_right_distance_sensor; visual box size=0.02 0.02 0.02
Joints:
- removed joint base_to_front_distance_sensor
- added joint base_to_front_left_distance_sensor: type fixed, parent /base_link, child /front_left_distance_sensor, origin xyz=0.22 0.09 -0.04 rpy=0 0 0
- added joint base_to_front_right_distance_sensor: type fixed, parent /base_link, child /front_right_distance_sensor, origin xyz=0.22 -0.09 -0.04 rpy=0 0 0
- joint base_to_rear_distance_sensor: origin xyz=-0.27 0.0 -0.04 rpy=0 0 3.14159 -> xyz=-0.27 0.0 0.04 rpy=0 0 3.14159

Commit message: no message

File: holly_tf/holly.urdf (robot description, URDF)
Before this commit: robot holly, 18 links, 17 joints
Joints:
- joint base_to_front_left_distance_sensor: origin xyz=0.22 0.09 -0.04 rpy=0 0 0 -> xyz=0.22 -0.09 -0.04 rpy=0 0 0
- joint base_to_front_right_distance_sensor: origin xyz=0.22 -0.09 -0.04 rpy=0 0 0 -> xyz=0.22 0.09 -0.04 rpy=0 0 0

Commit message: model reconfig

File: holly_tf/holly.urdf (robot description, URDF)
Before this commit: robot holly, 18 links, 17 joints
Links:
- removed link /laserscan_frame
- added link /kinect_frame
- added link /laserscan_sensor; visual box size=0.05 0.05 0.05
Joints:
- joint base_to_front_left_distance_sensor: origin xyz=0.22 -0.09 -0.04 rpy=0 0 0 -> xyz=0.25 -0.09 0.0 rpy=0 0 0
- joint base_to_front_right_distance_sensor: origin xyz=0.22 0.09 -0.04 rpy=0 0 0 -> xyz=0.25 0.09 0.0 rpy=0 0 0
- joint base_to_kinect_sensor: origin xyz=0.25 0.0 0.34 rpy=0 0.261799 0 -> xyz=0.2 0.0 0.05 rpy=0 0 0
- joint base_to_laserscan_sensor: child /laserscan_frame -> /laserscan_sensor; origin xyz=0.32 0.0 0.0 rpy=0 0 0 -> xyz=0.2 0 0.1 rpy=0 0 0

Commit message: rename the laserscan frame

File: holly_tf/holly.urdf (robot description, URDF)
Before this commit: robot holly, 19 links, 17 joints
Links:
- removed link /kinect_frame
- added link /kinect_laserscan_frame
Joints:
- added joint base_to_kinect_laserscan_frame: type fixed, parent /base_link, child /kinect_laserscan_frame, origin xyz=0.32 0.0 0.0 rpy=0 0 0

Commit message: sensor is tilted

File: holly_tf/holly.urdf (robot description, URDF)
Before this commit: robot holly, 19 links, 18 joints
Joints:
- joint base_to_kinect_sensor: origin xyz=0.2 0.0 0.05 rpy=0 0 0 -> xyz=0.2 0.0 0.05 rpy=0 -0.05 0

Commit message: no message

File: holly_tf/holly.urdf (robot description, URDF)
Before this commit: robot holly, 19 links, 18 joints
Joints:
- joint base_to_kinect_sensor: origin xyz=0.2 0.0 0.05 rpy=0 -0.05 0 -> xyz=0.2 0.0 0.05 rpy=0 -0.055 0

Commit message: rotate the laserscan sensor

File: holly_tf/holly.urdf (robot description, URDF)
Before this commit: robot holly, 19 links, 18 joints
Joints:
- joint base_to_laserscan_sensor: origin xyz=0.2 0 0.1 rpy=0 0 0 -> xyz=0.2 0 0.1 rpy=0 0 3.14159

Commit message: rename sensor

File: holly_tf/holly.urdf (robot description, URDF)
Before this commit: robot holly, 19 links, 18 joints
Links:
- removed link /laserscan_sensor
- added link /rplidar_sensor; visual box size=0.05 0.05 0.05
Joints:
- removed joint base_to_laserscan_sensor
- added joint base_to_rplidar_sensor: type fixed, parent /base_link, child /rplidar_sensor, origin xyz=0.2 0 0.1 rpy=0 0 0

Commit message: model tweaks

File: holly_tf/holly.urdf (robot description, URDF)
Before this commit: robot holly, 19 links, 18 joints
Joints:
- joint base_to_base_footprint: origin xyz=0 0 -0.2 -> xyz=0 0 -0.21
- joint base_to_kinect_laserscan_frame: origin xyz=0.32 0.0 0.0 rpy=0 0 0 -> xyz=0.24 0.0 0.0 rpy=0 0 0
- joint base_to_kinect_sensor: origin xyz=0.2 0.0 0.05 rpy=0 -0.055 0 -> xyz=0.24 0.0 0.05 rpy=0 -0.055 0
- joint base_to_rplidar_sensor: origin xyz=0.2 0 0.1 rpy=0 0 0 -> xyz=0.15 0 0.16 rpy=0 0 0

Commit message: Rotate the lidar sensor

File: holly_tf/holly.urdf (robot description, URDF)
Before this commit: robot holly, 19 links, 18 joints
Joints:
- joint base_to_rplidar_sensor: origin xyz=0.15 0 0.16 rpy=0 0 0 -> xyz=0.15 0 0.16 rpy=0 0 3.14159
